File: pcb/main/main.kicad_sch (KiCad schematic)
At the start: 90 parts, among them J1 USB_C, J2 Conn_01x03, J3 Conn_01x24, J4 Conn_01x12, J5 Conn_01x03, J6 Micro_SD_Card, J7 Conn_01x01, J8 Conn_01x02, SW1 SW_Push, U1 RP2350_60QFN, U2 W25Q128JVS, U3 NCP1117-3.3_SOT223, U4 ICM-42688-P, U5 BMP280, U6 MP9447, U7 ACS758xCB-100B-PSF, U8 NCP1117-3.3_SOT223, Y1 ABM8-272-T3

Commit message: progress
Parts:
- removed C27: 33n, Capacitor_SMD:C_0402_1005Metric, symbol Device:C
- removed C28, C32: 100n, Capacitor_SMD:C_0402_1005Metric, symbol Device:C
- removed C29: 390p, Capacitor_SMD:C_0402_1005Metric, symbol Device:C
- removed C30, C31: 22u, Capacitor_SMD:C_0805_2012Metric, symbol Device:C
- removed D2: PMEG4050EP, Diode_SMD:D_SOD-128, symbol Diode:PMEG4050EP
- removed D4: PESD1IVN27-AX, Diode_SMD:D_SOD-323F, symbol Device:D_TVS
- removed J5: Conn_01x03, symbol Connector_Generic:Conn_01x03
- removed L2: 10u, Inductor_SMD:L_1008_2520Metric, symbol Device:L
- removed R24: 7k, Resistor_SMD:R_0402_1005Metric, symbol Device:R
- removed U6: MP9447, toto_flight:QFN25_MP9447_MNP, symbol toto_flight:MP9447
- removed U7: ACS758xCB-100B-PSF, Sensor_Current:Allegro_CB_PSF, symbol Sensor_Current:ACS758xCB-100B-PSF
- added D2: PMEG2020EH, Diode_SMD:D_SOD-123F, symbol Diode:PMEG2020EH
- added D4: PESD5Z5.0, Diode_SMD:D_SOD-523, symbol Device:D_Schottky
- added J5: Conn_01x06, symbol Connector_Generic:Conn_01x06
- added RN1, RN2: 47, symbol Device:R_Pack08
- added RN3: 33, symbol Device:R_Pack02
- added U6: USBLC6-2SC6, Package_TO_SOT_SMD:SOT-23-6, symbol Power_Protection:USBLC6-2SC6
- added U7, U9: TLV2372, symbol Amplifier_Operational:TLV2372
- C12, C13: footprint toto_flight:C_0402_1005Metric_small_pads -> main:C_0402_1005Metric_small_pads
- C25: value 10u -> 10nF; footprint Capacitor_SMD:C_0805_2012Metric -> (none)
- C26: value 1u -> 10nF; footprint Capacitor_SMD:C_0402_1005Metric -> (none)
- J1: footprint toto_flight:YTC-TC8S-126 -> main:YTC-TC8S-126; symbol toto_flight:USB_C -> main:USB_C
- J6: footprint toto_flight:MOLEX_104031-0811 -> main:MOLEX_104031-0811; symbol toto_flight:Micro_SD_Card -> main:Micro_SD_Card
- L1: footprint toto_flight:L_pol_2016 -> main:L_pol_2016
- R16: value 499k -> 47; footprint Resistor_SMD:R_0402_1005Metric -> (none)
- R17: value 100k -> 7K; footprint Resistor_SMD:R_0402_1005Metric -> (none)
- R18: value 845k -> 10K; footprint Resistor_SMD:R_0805_2012Metric -> (none)
- R19: value 10k -> 10K; footprint Resistor_SMD:R_0402_1005Metric -> (none)
- R20: value 53.6k -> 47; footprint Resistor_SMD:R_0402_1005Metric -> (none)
- R21: value 100k -> 100; footprint Resistor_SMD:R_0402_1005Metric -> (none)
- R22, R23: value 100k -> 47; footprint Resistor_SMD:R_0402_1005Metric -> (none)
- R7: value 5.1k -> 47K; footprint Capacitor_SMD:C_0402_1005Metric -> (none)
- U1: footprint toto_flight:RP2350-QFN-60-1EP_7x7_P0.4mm_EP3.4x3.4mm_ThermalVias -> main:RP2350-QFN-60-1EP_7x7_P0.4mm_EP3.4x3.4mm_ThermalVias; symbol toto_flight:RP2350_60QFN -> main:RP2350_60QFN
- U4: footprint toto_flight:LGA14_2P5X3X0P91_TDK -> main:LGA14_2P5X3X0P91_TDK; symbol toto_flight:ICM-42688-P -> main:ICM-42688-P
- U5: footprint toto_flight:BMP280 -> main:BMP280
Connections:
- net VBAT is gone; now on net GP29: R23.2
- net +3V3: no longer C22.1, R27.1, U4.5 (VDDIO)
- net +5V: now also D2.1 (K)
- net 3v3_IMU: now also C22.1, R27.1, U4.5 (VDDIO)
- net 5V_BEC: now also D2.2 (A), D4.1 (K), J5.1 (Pin_1), J5.6 (Pin_6); no longer R20.1
- net GND: now also C26.1, R17.1, D4.2 (A), J5.2 (Pin_2), J5.5 (Pin_5), U6.2 (GND); no longer C26.2, R17.2, R21.2, R7.2
- net GP0: now also RN1.1 (R1.1); no longer J3.3 (Pin_3)
- net GP1: now also RN1.2 (R2.1); no longer J3.4 (Pin_4)
- net GP10: now also RN1.7 (R7.1); no longer J3.15 (Pin_15)
- net GP11: now also RN1.8 (R8.1); no longer J3.16 (Pin_16)
- net GP16: now also RN2.1 (R1.1); no longer J3.19 (Pin_19)
- net GP17: now also RN2.2 (R2.1); no longer J3.20 (Pin_20)
- net GP18: now also RN2.3 (R3.1); no longer J3.23 (Pin_23)
- net GP19: now also RN2.4 (R4.1); no longer J3.24 (Pin_24)
- net GP20: now also RN2.5 (R5.1); no longer J4.1 (Pin_1)
- net GP21: now also RN2.6 (R6.1); no longer J4.4 (Pin_4)
- net GP22: now also RN2.7 (R7.1); no longer J4.7 (Pin_7)
- net GP23: now also RN2.8 (R8.1); no longer J4.10 (Pin_10)
- net GP24: now also R16.1; no longer J7.1 (Pin_1)
- net GP26: now also U7.1, U7.2 (-); no longer R23.1
- net GP27: now also U9.1, U9.2 (-); no longer R21.1, R22.2
- net GP28: now also R22.1; no longer J8.1 (Pin_1)
- net GP29: no longer J8.2 (Pin_2)
- net GP8: now also RN1.5 (R5.1); no longer J3.11 (Pin_11)
- net GP9: now also RN1.6 (R6.1); no longer J3.12 (Pin_12)
- net I2C0_SCL: now also RN1.4 (R4.1); no longer J3.8 (Pin_8)
- net I2C0_SDA: now also RN1.3 (R3.1); no longer J3.7 (Pin_7)
- net SWCLK: now also RN3.3 (R2.2); no longer J2.1 (Pin_1)
- net SWD: now also RN3.4 (R1.2); no longer J2.3 (Pin_3)
- net USB_D+: now also U6.4 (I/O2); no longer J1.B6 (D+)
- net USB_D-: now also U6.6 (I/O1); no longer J1.B7 (D-)
- net VBUS: now also U6.5 (VBUS)
- net at R16.2: now also J7.1 (Pin_1)
- net CURR_A: now reaches R18.2
- net CURR_A: now also J5.4 (Pin_4)
- net at R20.2: now also C25.2, U9.3 (+); no longer R19.1
- net VBAT_A: now reaches R7.1
- net VBAT_A: now also J5.3 (Pin_3)
- removed net VBAT_P: C25.2, R16.1
- new net: J3.15 (Pin_15), RN1.10 (R7.2)
- new net: J3.12 (Pin_12), RN1.11 (R6.2)
- new net: J3.11 (Pin_11), RN1.12 (R5.2)
- new net: J3.8 (Pin_8), RN1.13 (R4.2)
- new net: J3.7 (Pin_7), RN1.14 (R3.2)
- new net: J3.4 (Pin_4), RN1.15 (R2.2)
- new net: J3.3 (Pin_3), RN1.16 (R1.2)
- new net: J3.16 (Pin_16), RN1.9 (R8.2)
- new net: J1.B7 (D-), U6.1 (I/O1)
- new net: J1.B6 (D+), U6.3 (I/O2)
- new net: J8.1 (Pin_1), R22.2
- new net: J8.2 (Pin_2), R23.1
- new net: J4.1 (Pin_1), RN2.12 (R5.2)
- new net: J4.10 (Pin_10), RN2.9 (R8.2)
- new net: J4.4 (Pin_4), RN2.11 (R6.2)
- new net: J4.7 (Pin_7), RN2.10 (R7.2)
- new net: R19.1, R20.1
- new net: C26.2, R21.2, U7.3 (+)
- new net: J2.3 (Pin_3), RN3.1 (R1.1)
- new net: J2.1 (Pin_1), RN3.2 (R2.1)
- new net: R17.2, R21.1, R7.2
- new net: J3.24 (Pin_24), RN2.13 (R4.2)
- new net: J3.23 (Pin_23), RN2.14 (R3.2)
- new net: J3.20 (Pin_20), RN2.15 (R2.2)
- new net: J3.19 (Pin_19), RN2.16 (R1.2)
Other:
- note added: "Connector"
- note added: "USB C AND POWER"
- note added: "VBAT AND CURR"
- note removed: "BEC"
- note removed: "Protection and Sensors"
- note removed: "USB C"
- note removed: "VBAT"
- moved on the sheet: C1, C10, C11, C12, C13, C14, C15, C16, C17, C18, C19, C2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
