File: pcb/power/toto_flight_old.kicad_pcb (KiCad board)
At the start: 2 copper layers, 43.6 x 53.4 mm, 58 parts, among them J1 USB_C, J2 Conn_01x03, J3 Conn_01x16, J4 Conn_01x15, J5 Conn_01x02, J6 Micro_SD_Card, J7 Conn_01x08, J8 Conn_01x04, SW1 SW_Push, U1 RP2350_60QFN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

Commit message: progress
Parts:
- C12, C13: footprint toto_flight:C_0402_1005Metric_small_pads -> power:C_0402_1005Metric_small_pads
- J1: footprint toto_flight:USB_C_017 -> power:USB_C_017
- J3: footprint toto_flight:gpio_pads -> power:gpio_pads
- J4: footprint toto_flight:pwm_pins -> power:pwm_pins
- J5: footprint toto_flight:esc_power_pads -> power:esc_power_pads
- J6: footprint toto_flight:MOLEX_104031-0811 -> power:MOLEX_104031-0811
- J7: footprint toto_flight:gpio_2_pads -> power:gpio_2_pads
- J8: footprint toto_flight:analog_pads -> power:analog_pads
- L1: footprint toto_flight:L_pol_2016 -> power:L_pol_2016
- U1: footprint toto_flight:RP2350-QFN-60-1EP_7x7_P0.4mm_EP3.4x3.4mm_ThermalVias -> power:RP2350-QFN-60-1EP_7x7_P0.4mm_EP3.4x3.4mm_ThermalVias
- U4: footprint toto_flight:LGA14_2P5X3X0P91_TDK -> power:LGA14_2P5X3X0P91_TDK
- U5: footprint toto_flight:BMP280 -> power:BMP280
