File: pcb/fc_board/toto_flight_old.kicad_pcb (KiCad board)
At the start: 2 copper layers, 43.6 x 53.4 mm, 58 parts, among them J1 USB_C, J2 Conn_01x03, J3 Conn_01x16, J4 Conn_01x15, J5 Conn_01x02, J6 Micro_SD_Card, J7 Conn_01x08, J8 Conn_01x04, SW1 SW_Push, U1 RP2350_60QFN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

Commit message: rename pcbs
Parts:
- C12, C13: footprint main:C_0402_1005Metric_small_pads -> fc_board:C_0402_1005Metric_small_pads
- J1: footprint main:USB_C_017 -> fc_board:USB_C_017
- J3: footprint main:gpio_pads -> fc_board:gpio_pads
- J4: footprint main:pwm_pins -> fc_board:pwm_pins
- J5: footprint main:esc_power_pads -> fc_board:esc_power_pads
- J6: footprint main:MOLEX_104031-0811 -> fc_board:MOLEX_104031-0811
- J7: footprint main:gpio_2_pads -> fc_board:gpio_2_pads
- J8: footprint main:analog_pads -> fc_board:analog_pads
- L1: footprint main:L_pol_2016 -> fc_board:L_pol_2016
- U1: footprint main:RP2350-QFN-60-1EP_7x7_P0.4mm_EP3.4x3.4mm_ThermalVias -> fc_board:RP2350-QFN-60-1EP_7x7_P0.4mm_EP3.4x3.4mm_ThermalVias
- U4: footprint main:LGA14_2P5X3X0P91_TDK -> fc_board:LGA14_2P5X3X0P91_TDK
- U5: footprint main:BMP280 -> fc_board:BMP280
