File: pcb/fc_board/fc_board.kicad_sch (KiCad schematic)
At the start: 86 parts, among them J1 USB_C, J2 Conn_01x03, J3 Conn_01x24, J4 Conn_01x12, J5 Conn_01x06, J6 Micro_SD_Card, J7 Conn_01x01, J8 Conn_01x02, SW1 SW_Push, U1 RP2350_60QFN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

Commit message: rename pcbs
Parts:
- C12, C13: footprint main:C_0402_1005Metric_small_pads -> fc_board:C_0402_1005Metric_small_pads
- J1: footprint main:YTC-TC8S-126 -> fc_board:YTC-TC8S-126; symbol main:USB_C -> fc_board:USB_C
- J6: footprint main:MOLEX_104031-0811 -> fc_board:MOLEX_104031-0811; symbol main:Micro_SD_Card -> fc_board:Micro_SD_Card
- L1: footprint main:L_pol_2016 -> fc_board:L_pol_2016
- U1: footprint main:RP2350-QFN-60-1EP_7x7_P0.4mm_EP3.4x3.4mm_ThermalVias -> fc_board:RP2350-QFN-60-1EP_7x7_P0.4mm_EP3.4x3.4mm_ThermalVias; symbol main:RP2350_60QFN -> fc_board:RP2350_60QFN
- U4: footprint main:LGA14_2P5X3X0P91_TDK -> fc_board:LGA14_2P5X3X0P91_TDK; symbol main:ICM-42688-P -> fc_board:ICM-42688-P
- U5: footprint main:BMP280 -> fc_board:BMP280

Commit message: fc_board: More schematic progress
Parts:
- removed C19, C20, C23, C24: 100n, Capacitor_SMD:C_0402_1005Metric, symbol Device:C
- removed C21: 2.2u, Capacitor_SMD:C_0402_1005Metric, symbol Device:C
- removed C22: 10n, Capacitor_SMD:C_0402_1005Metric, symbol Device:C
- removed C25, C26: 10nF, symbol Device:C
- removed C33, C34: 10u, Capacitor_SMD:C_0805_2012Metric, symbol Device:C
- removed D2, D3: PMEG2020EH, Diode_SMD:D_SOD-123F, symbol Diode:PMEG2020EH
- removed D4, D5: PESD5Z5.0, Diode_SMD:D_SOD-523, symbol Device:D_Schottky
- removed J1: USB_C, fc_board:YTC-TC8S-126, symbol fc_board:USB_C
- removed J2: Conn_01x03, Connector_PinHeader_2.54mm:PinHeader_1x03_P2.54mm_Vertical, symbol Connector_Generic:Conn_01x03
- removed J3: Conn_01x24, symbol Connector_Generic:Conn_01x24
- removed J4: Conn_01x12, symbol Connector_Generic:Conn_01x12
- removed J5: Conn_01x06, symbol Connector_Generic:Conn_01x06
- removed J6: Micro_SD_Card, fc_board:MOLEX_104031-0811, symbol fc_board:Micro_SD_Card
- removed J7: Conn_01x01, symbol Connector_Generic:Conn_01x01
- removed J8: Conn_01x02, symbol Connector_Generic:Conn_01x02
- removed R10, R11, R12, R13: 50k, Resistor_SMD:R_0402_1005Metric, symbol Device:R
- removed R14, R15: 2.2k, Resistor_SMD:R_0402_1005Metric, symbol Device:R
- removed R16, R20, R22, R23: 47, symbol Device:R
- removed R17: 7K, symbol Device:R
- removed R18, R19: 10K, symbol Device:R
- removed R21: 100, symbol Device:R
- removed R27: 10k, Resistor_SMD:R_0402_1005Metric, symbol Device:R
- removed R7: 47K, symbol Device:R
- removed R8: 5.1k, Capacitor_SMD:C_0402_1005Metric, symbol Device:R
- removed RN1, RN2: 47, symbol Device:R_Pack08
- removed RN3: 33, symbol Device:R_Pack02
- removed U4: ICM-42688-P, fc_board:LGA14_2P5X3X0P91_TDK, symbol fc_board:ICM-42688-P
- removed U5: BMP280, fc_board:BMP280, symbol Sensor_Pressure:BMP280
- removed U6: USBLC6-2SC6, Package_TO_SOT_SMD:SOT-23-6, symbol Power_Protection:USBLC6-2SC6
- removed U7, U9: TLV2372, symbol Amplifier_Operational:TLV2372
- removed U8: NCP1117-3.3_SOT223, Package_TO_SOT_SMD:SOT-223-3_TabPin2, symbol Regulator_Linear:NCP1117-3.3_SOT223
- R9: value 470 -> 1k
Connections:
- net +3V3: now also R6.2; no longer R6.1
- net GND: now also SW1.2; no longer SW1.1
- net at R5.1: now also SW1.1; no longer SW1.2
- net I2C0_SCL renamed GP7
- net I2C0_SDA renamed GP6
- net RUN: no longer names the net of U1.26 (RUN)
- net RUN: now also R6.1; no longer R6.2
- net SPI0_CLK renamed GP2
- net SPI0_CS_IMU renamed GP5
- net SPI0_RX renamed GP4
- net SPI0_TX renamed GP3
- net SPI1_CLK renamed GP14
- net SPI1_CS_SD_CARD renamed GP13
- net SPI1_RX renamed GP12
- net SPI1_TX renamed GP15
- net USB_D+ renamed USB-C and POWER/USB_D+
- net USB_D- renamed USB-C and POWER/USB_D-
- no-connect marks 4 -> 0
Other:
- added sheet Connectors (connectors.kicad_sch)
- added sheet Peripherals (peripherals.kicad_sch)
- added sheet USB-C and POWER (usb_c_and_power.kicad_sch)
- note added: "BOOT SELECT"
- note added: "MAIN"
- note removed: "ANALOG"
- note removed: "BARO"
- note removed: "Boot Select"
- note removed: "Connector"
- note removed: "GPIO"
- note removed: "IMU"
- note removed: "PWM"
- note removed: "RUN"
- note removed: "SWD"
- note removed: "USB C AND POWER"
- note removed: "VBAT AND CURR"
- moved on the sheet: C1, C10, C11, C12, C13, C14, C15, C16, C17, C18, C2, C3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
