File: pcb/power_board/power_board.kicad_sch (KiCad schematic)
At the start: 17 parts, among them J1 Conn_01x06, U6 MP9447, U7 ACS758xCB-100B-PSF

Commit message: rename pcbs
Parts:
- U6: footprint power:QFN25_MP9447_MNP -> power_board:QFN25_MP9447_MNP; symbol power:MP9447 -> power_board:MP9447
Changed lines of the file:
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@@
 		)
 		(instances
-			(project "power"
+			(project "power_board"
 				(path "/0259efb7-694a-4ce2-9998-fdf65c8a3c90"
 					(reference "D4")
@@
 	)
 	(symbol
-		(lib_id "power:5V_BEC")
+		(lib_id "power_board:5V_BEC")
 		(at 168.91 53.34 90)
 		(unit 1)
@@
 		)
 		(instances
-			(project "power"
+			(project "power_board"
 				(path "/0259efb7-694a-4ce2-9998-fdf65c8a3c90"
 					(reference "#PWR01")
@@
 		)
 		(instances
-			(project "power"
+			(project "power_board"
 				(path "/0259efb7-694a-4ce2-9998-fdf65c8a3c90"
 					(reference "C26")
@@
 		)
 		(instances
-			(project "power"
+			(project "power_board"
 				(path "/0259efb7-694a-4ce2-9998-fdf65c8a3c90"
 					(reference "C30")
@@
 	)
 	(symbol
-		(lib_id "power:GND")
+		(lib_id "power_board:GND")
 		(at 55.88 110.49 270)
 		(unit 1)
@@
 		)
 		(instances
-			(project "power"
+			(project "power_board"
 				(path "/0259efb7-694a-4ce2-9998-fdf65c8a3c90"
 					(reference "#PWR058")
@@
 	)
 	(symbol
-		(lib_id "power:GND")
+		(lib_id "power_board:GND")
 		(at 128.27 133.35 0)
 		(unit 1)
@@
 		)
 		(instances
-			(project "power"
+			(project "power_board"
 				(path "/0259efb7-694a-4ce2-9998-fdf65c8a3c90"
 					(reference "C29")
@@
 	)
 	(symbol
-		(lib_id "power:GND")
+		(lib_id "power_board:GND")
 		(at 48.26 66.04 0)
 		(unit 1)
@@
 		)
 		(instances
-			(project "power"
+			(project "power_board"
 				(path "/0259efb7-694a-4ce2-9998-fdf65c8a3c90"
 					(reference "#PWR062")
@@
 	)
 	(symbol
-		(lib_id "power:VBAT_P")
+		(lib_id "power_board:VBAT_P")
 		(at 78.74 55.88 90)
 		(unit 1)
@@
 		)
 		(instances
-			(project "power"
+			(project "power_board"
 				(path "/0259efb7-694a-4ce2-9998-fdf65c8a3c90"
 					(reference "#PWR083")
@@
 	)
 	(symbol
-		(lib_id "power:MP9447")
+		(lib_id "power_board:MP9447")
 		(at 74.93 95.25 0)
 		(unit 1)
@@
 			)
 		)
-		(property "Footprint" "power:QFN25_MP9447_MNP"
+		(property "Footprint" "power_board:QFN25_MP9447_MNP"
 			(at 74.93 95.25 0)
 			(effects
@@
 	)
 	(symbol
-		(lib_id "power:GND")
+		(lib_id "power_board:GND")
 		(at 44.45 106.68 0)
 		(unit 1)
@@
 	)
 	(symbol
-		(lib_id "power:VBAT_P")
+		(lib_id "power_board:VBAT_P")
 		(at 26.67 93.98 90)
 		(unit 1)
@@
 	)
 	(symbol
-		(lib_id "power:GND")
+		(lib_id "power_board:GND")
 		(at 88.9 60.96 0)
 		(unit 1)
@@
 		)
 		(instances
-			(project "power"
+			(project "power_board"
 				(path "/0259efb7-694a-4ce2-9998-fdf65c8a3c90"
 					(reference "R18")
@@
 		)
 		(instances
-			(project "power"
+			(project "power_board"
 				(path "/0259efb7-694a-4ce2-9998-fdf65c8a3c90"
 					(reference "R20")
@@
 	(symbol
 		(lib_name "5V_BEC_1")
-		(lib_id "power:5V_BEC")
+		(lib_id "power_board:5V_BEC")
 		(at 88.9 43.18 0)
 		(unit 1)
@@
 	)
 	(symbol
-		(lib_id "power:5V_BEC")
+		(lib_id "power_board:5V_BEC")
 		(at 168.91 66.04 90)
 		(unit 1)
@@
 		)
 		(instances
-			(project "power"
+			(project "power_board"
 				(path "/0259efb7-694a-4ce2-9998-fdf65c8a3c90"
 					(reference "#PWR02")
@@
 		)
 		(instances
-			(project "power"
+			(project "power_board"
 				(path "/0259efb7-694a-4ce2-9998-fdf65c8a3c90"
 					(reference "R17")
@@
 	)
 	(symbol
-		(lib_id "power:GND")
+		(lib_id "power_board:GND")
 		(at 62.23 83.82 180)
 		(unit 1)
@@
 		)
 		(instances
-			(project "power"
+			(project "power_board"
 				(path "/0259efb7-694a-4ce2-9998-fdf65c8a3c90"
 					(reference "#PWR056")
@@
 		)
 		(instances
-			(project "power"
+			(project "power_board"
 				(path "/0259efb7-694a-4ce2-9998-fdf65c8a3c90"
 					(reference "R19")
@@
 		)
 		(instances
-			(project "power"
+			(project "power_board"
 				(path "/0259efb7-694a-4ce2-9998-fdf65c8a3c90"
 					(reference "C28")
@@
 	)
 	(symbol
-		(lib_id "power:GND")
+		(lib_id "power_board:GND")
 		(at 34.29 104.14 0)
 		(unit 1)
@@
 		)
 		(instances
-			(project "power"
+			(project "power_board"
 				(path "/0259efb7-694a-4ce2-9998-fdf65c8a3c90"
 					(reference "#PWR054")
@@
 	)
 	(symbol
-		(lib_id "power:VBAT")
+		(lib_id "power_board:VBAT")
 		(at 35.56 50.8 90)
 		(unit 1)
@@
 		)
 		(instances
-			(project "power"
+			(project "power_board"
 				(path "/0259efb7-694a-4ce2-9998-fdf65c8a3c90"
 					(reference "C31")
@@
 	)
 	(symbol
-		(lib_id "power:5V_BEC")
+		(lib_id "power_board:5V_BEC")
 		(at 165.1 104.14 270)
 		(unit 1)
@@
 		)
 		(instances
-			(project "power"
+			(project "power_board"
 				(path "/0259efb7-694a-4ce2-9998-fdf65c8a3c90"
 					(reference "C27")
