File: pcb/peripherals.kicad_sch (KiCad schematic)
At the start: 18 parts, among them J6 Micro_SD_Card, U4 ICM-42688-P, U5 BMP280, U8 NCP1117-3.3_SOT223

Commit message: Huge huge refactor and use pico
Parts:
- removed C33, C34: 10u, Capacitor_SMD:C_0805_2012Metric, symbol Device:C
- removed U8: NCP1117-3.3_SOT223, Package_TO_SOT_SMD:SOT-223-3_TabPin2, symbol Regulator_Linear:NCP1117-3.3_SOT223
- added C10, C11, C7: 100n, symbol Device:C
- added U3: TPS79133DBVR, toto_fc:TPS79133DBVR, symbol toto_fc:TPS79133DBVR
- C12: renamed from C23; footprint Capacitor_SMD:C_0402_1005Metric -> (none)
- C13: renamed from C24; footprint Capacitor_SMD:C_0402_1005Metric -> (none)
- C14: renamed from C19; footprint Capacitor_SMD:C_0402_1005Metric -> (none)
- C8: renamed from C22; footprint Capacitor_SMD:C_0402_1005Metric -> (none)
- C9: renamed from C27; footprint Capacitor_SMD:C_0402_1005Metric -> (none)
- J11: renamed from J6; footprint fc_board:MOLEX_104031-0811 -> toto_fc:MOLEX_104031-0811; symbol fc_board:Micro_SD_Card -> toto_fc:Micro_SD_Card
- R10: renamed from R13; footprint Resistor_SMD:R_0402_1005Metric -> (none)
- R11: renamed from R12; footprint Resistor_SMD:R_0402_1005Metric -> (none)
- R12: renamed from R11; footprint Resistor_SMD:R_0402_1005Metric -> (none)
- R13: renamed from R10; footprint Resistor_SMD:R_0402_1005Metric -> (none)
- R7: renamed from R27; footprint Resistor_SMD:R_0402_1005Metric -> (none)
- R8: renamed from R14; footprint Resistor_SMD:R_0402_1005Metric -> (none)
- R9: renamed from R15; footprint Resistor_SMD:R_0402_1005Metric -> (none)
- U2: renamed from U4; footprint LGA14_2P5X3X0P91_TDK -> toto_fc:ICM-42688-P; symbol fc_board:ICM-42688-P -> toto_fc:ICM-42688-P
- U4: renamed from U5; footprint fc_board:BMP280 -> toto_fc:BMP280; now fitted
Connections:
- net +3V3: no longer R8.2, R9.2
- net +5V: now also C7.1, U3.1 (IN)
- net GND: now also U2.11 (RESV_GND), U2.7 (RESV_GND), C10.2, C11.2, C7.2, U3.2 (GND), U3.3 (EN)
- net 3v3_IMU renamed 3v3_SENSOR
- net 3v3_SENSOR: now also R8.2, R9.2, C11.1, U3.5 (OUT)
- net I2C0_SCL renamed BARO_I2C_SCL
- net I2C0_SDA renamed BARO_I2C_SDA
- net SPI0_CLK renamed IMU_SPI_CLK
- net SPI0_CS_IMU renamed IMU_SPI_CS
- net SPI0_MISO renamed IMU_SPI_MISO
- net SPI0_MOSI renamed IMU_SPI_MOSI
- net SPI1_CLK renamed SD_CARD_SPI_CLK
- net SPI1_CS_SD_CARD renamed SD_CARD_SPI_CS
- net SPI1_MISO renamed SD_CARD_SPI_MISO
- net SPI1_MOSI renamed SD_CARD_SPI_MOSI
- new net: C10.1, U3.4 (BYPASS)
- new net: U2.10 (RESV), U2.2 (RESV), U2.3 (RESV)
- now unconnected: U2.4 (INT1/INT), U2.9 (INT2/FSYNC/CLKIN)
- no-connect marks 1 -> 4
Other:
- note added: "SENSOR LDO"
- moved on the sheet: C12, C13, C14, C8, C9, R7, R8, R9

Commit message: More pcb work
Parts:
- removed U4: BMP280, toto_fc:BMP280, symbol Sensor_Pressure:BMP280
- added U4: BMP390, toto_fc:BMP390, symbol toto_fc:BMP390
- C10: renamed from C9; footprint (none) -> Capacitor_SMD:C_0603_1608Metric
- C11: renamed from C10; footprint (none) -> Capacitor_SMD:C_0603_1608Metric
- C12: renamed from C11; footprint (none) -> Capacitor_SMD:C_0603_1608Metric
- C13: renamed from C12; footprint (none) -> Capacitor_SMD:C_0603_1608Metric
- C14: renamed from C13; footprint (none) -> Capacitor_SMD:C_0603_1608Metric
- C15: renamed from C14; footprint (none) -> Capacitor_SMD:C_0603_1608Metric
- C8: renamed from C7; footprint (none) -> Capacitor_SMD:C_0603_1608Metric
- C9: renamed from C8; footprint (none) -> Capacitor_SMD:C_0603_1608Metric
- R10, R11, R12, R13, R7: footprint (none) -> Resistor_SMD:R_0603_1608Metric
- R8, R9: value 2.2k -> 4.7k; footprint (none) -> Resistor_SMD:R_0603_1608Metric
Connections:
- net 3v3_SENSOR: now also U4.1 (VDDIO), U4.10 (VDD), U4.6 (CSB)
- net BARO_I2C_SCL: now also U4.2 (SCK)
- net BARO_I2C_SDA: now also U4.4 (SDI)
- net GND: now also U4.3 (GND), U4.5 (SDO), U4.8 (GND), U4.9 (GND)
- no-connect marks 4 -> 5
Other:
- moved on the sheet: C13, C14, R8, R9
