File: pcb/toto_fc.kicad_pcb (KiCad board)
At the start: 4 copper layers, 36.5 x 56 mm, 0 parts

Commit message: More pcb work
Parts:
- added A1: RaspberryPi_Pico, Module:RaspberryPi_Pico_SMD_HandSolder, B.Cu at (45.2, 66.0)
- added C1: 10u, Capacitor_SMD:C_0805_2012Metric, F.Cu at (50.5, 83.5)
- added C10: 2.2u, Capacitor_SMD:C_0603_1608Metric, F.Cu at (46.8, 51.0)
- added C11: 100n, Capacitor_SMD:C_0603_1608Metric, F.Cu at (45.5, 57.5)
- added C12: 100n, Capacitor_SMD:C_0603_1608Metric, F.Cu at (39.5, 56.5)
- added C13: 100n, Capacitor_SMD:C_0603_1608Metric, F.Cu at (42.5, 50.5)
- added C14: 100n, Capacitor_SMD:C_0603_1608Metric, F.Cu at (40.5, 52.5)
- added C15: 100n, Capacitor_SMD:C_0603_1608Metric, F.Cu at (48.0, 61.0)
- added C2: 100n, Capacitor_SMD:C_0603_1608Metric, F.Cu at (49.0, 85.5)
- added C3: 10u, Capacitor_SMD:C_0805_2012Metric, F.Cu at (47.0, 79.0)
- added C4: 33p, Capacitor_SMD:C_0603_1608Metric, F.Cu at (44.0, 85.2)
- added C5: 33u, Capacitor_SMD:C_0805_2012Metric, F.Cu at (39.5, 73.5)
- added C6: 33u, Capacitor_SMD:C_0805_2012Metric, F.Cu at (41.5, 73.6)
- added C7: 1u, Capacitor_SMD:C_0603_1608Metric, F.Cu at (39.5, 63.5)
- added C8: 100n, Capacitor_SMD:C_0603_1608Metric, F.Cu at (39.5, 58.5)
- added C9: 10n, Capacitor_SMD:C_0603_1608Metric, F.Cu at (46.8, 48.0)
- added D1: PESD1IVN27-AX, Diode_SMD:D_SOD-323F, B.Cu at (32.0, 76.0)
- added D2: PMEG2010EH, Diode_SMD:D_SOD-123F, F.Cu at (44.0, 68.5)
- added J1: Conn_01x02, toto_fc:vbat_pads, B.Cu at (29.0, 76.0)
- added J11: Micro_SD_Card, toto_fc:MOLEX_104031-0811, F.Cu at (55.5, 62.8)
- added J2: Conn_01x12, toto_fc:pwm_headers, B.Cu at (30.0, 52.2)
- added J3: Conn_01x03, Connector_PinHeader_2.54mm:PinHeader_1x03_P2.54mm_Vertical, B.Cu at (30.0, 63.1)
- added J4: Receiver Connector, Connector_JST:JST_GH_BM04B-GHS-TBT_1x04-1MP_P1.25mm_Vertical, B.Cu at (60.5, 63.5)
- added J5: GPS Connector, Connector_JST:JST_GH_BM06B-GHS-TBT_1x06-1MP_P1.25mm_Vertical, B.Cu at (60.5, 83.0)
- added J6: VTX Connector, Connector_JST:JST_GH_BM04B-GHS-TBT_1x04-1MP_P1.25mm_Vertical, B.Cu at (30.0, 86.5)
- added JP1: BEC_SJ, Jumper:SolderJumper-2_P1.3mm_Open_Pad1.0x1.5mm, F.Cu at (1.76, 74.2)
- added JP2: ESC_SJ, Jumper:SolderJumper-2_P1.3mm_Open_Pad1.0x1.5mm, F.Cu at (1.76, 77.7)
- added L1: 5.6u, toto_fc:F1C2-060606W-5R6M, F.Cu at (46.0, 74.6)
- added R1: 31.6k, Resistor_SMD:R_0603_1608Metric, F.Cu at (43.2, 79.7)
- added R10: 50k, Resistor_SMD:R_0603_1608Metric, F.Cu at (55.2, 54.3)
- added R11: 50k, Resistor_SMD:R_0603_1608Metric, F.Cu at (53.8, 54.3)
- added R12: 50k, Resistor_SMD:R_0603_1608Metric, F.Cu at (52.2, 54.3)
- added R13: 50k, Resistor_SMD:R_0603_1608Metric, F.Cu at (50.8, 54.3)
- added R2: 100k, Resistor_SMD:R_0603_1608Metric, F.Cu at (42.5, 82.2)
- added R3: 19.1k, Resistor_SMD:R_0603_1608Metric, F.Cu at (44.0, 82.2)
- added R4: 1k, Resistor_SMD:R_0603_1608Metric, F.Cu at (42.5, 85.2)
- added R5: 47K, Resistor_SMD:R_0603_1608Metric, F.Cu at (39.5, 66.5)
- added R6: 7K, Resistor_SMD:R_0603_1608Metric, F.Cu at (41.0, 63.5)
- added R7: 10k, Resistor_SMD:R_0603_1608Metric, F.Cu at (51.2, 50.8)
- added R8: 4.7k, Resistor_SMD:R_0603_1608Metric, F.Cu at (40.5, 46.5)
- added R9: 4.7k, Resistor_SMD:R_0603_1608Metric, F.Cu at (39.0, 46.5)
- added U1: LMR51450, toto_fc:LMR51450, F.Cu at (46.7, 82.6)
- added U2: ICM-42688-P, toto_fc:ICM-42688-P, F.Cu at (49.0, 48.9)
- added U3: TPS79133DBVR, toto_fc:TPS79133DBVR, F.Cu at (43.0, 57.5)
- added U4: BMP390, toto_fc:BMP390, F.Cu at (40.0, 49.5)
Other:
- board size 36.5 x 56 mm -> 37.5 x 53.5 mm
- copper layers 4 -> 2

Commit message: More work on the pcb
Parts:
- D1, J1: moved to F.Cu
- J4, J6: footprint Connector_JST:JST_GH_BM04B-GHS-TBT_1x04-1MP_P1.25mm_Vertical -> Connector_JST:JST_GH_SM04B-GHS-TB_1x04-1MP_P1.25mm_Horizontal; moved to F.Cu
- J5: footprint Connector_JST:JST_GH_BM06B-GHS-TBT_1x06-1MP_P1.25mm_Vertical -> Connector_JST:JST_GH_SM06B-GHS-TB_1x06-1MP_P1.25mm_Horizontal; moved to F.Cu
- moved JP1 39.1 mm to (40.5, 69.0), turned to 90 degrees
- moved JP2 36.8 mm to (37.0, 67.0)
- moved R10 16.2 mm to (44.0, 66.0), turned to 180 degrees
- moved J4 15.0 mm to (55.0, 49.5)
- moved R11 14.1 mm to (44.0, 64.5), turned to 180 degrees
- moved R12 9.74 mm to (44.0, 59.5), turned to 180 degrees
- moved J2 8.83 mm to (31.3, 43.5)
- moved R13 7.69 mm to (44.0, 58.0), turned to 180 degrees
- moved J5 6.26 mm to (55.0, 80.0)
- moved C4 5.41 mm to (38.8, 83.9), turned to 0 degrees
- moved D2 5.32 mm to (40.5, 64.5)
- moved R4 4.68 mm to (38.8, 82.4), turned to 0 degrees
- moved R6 4.44 mm to (36.8, 62.0), turned to 180 degrees
- moved C7 4.02 mm to (36.8, 60.5), turned to 0 degrees
- moved R5 4.02 mm to (36.8, 63.5), turned to 0 degrees
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Connections:
- net Net-(J3-Pin_2) renamed /ESC_BEC
- net Net-(JP1-A) renamed /ONBOARD_BEC
- J2 pad 1: GND -> /SERVO_PWM_1
- J2 pad 10: GND -> /SERVO_PWM_4
- J2 pad 12: /SERVO_PWM_4 -> GND
- J2 pad 3: /SERVO_PWM_1 -> GND
- J2 pad 4: GND -> /SERVO_PWM_2
- J2 pad 6: /SERVO_PWM_2 -> GND
- J2 pad 7: GND -> /SERVO_PWM_3
- J2 pad 9: /SERVO_PWM_3 -> GND
Other:
- board size 37.5 x 53.5 mm -> 32 x 53.5 mm
- board text added: "Toto FC Rev 0.2"

Commit message: more progress
Parts:
- removed D1: PESD1IVN27-AX, Diode_SMD:D_SOD-323F
- added CR1: D24V0S1U2TQ-7, toto_fc:SOD523, F.Cu at (32.0, 75.7)
- A1: footprint Module:RaspberryPi_Pico_SMD_HandSolder -> toto_fc:RaspberryPi_Pico_SMD_HandSolder
- moved C6 2.24 mm to (39.5, 74.0), turned to 90 degrees
- moved C5 1.00 mm to (37.5, 74.0), turned to 90 degrees
- moved JP1 0.55 mm to (40.5, 68.4)
- moved J4 0.40 mm to (54.9, 49.1)
Routing:
- net 3v3_SENSOR: track 0.00 -> 38.5 mm
- net /SERVO_PWM_3: track 0.00 -> 33.8 mm, vias 0 -> 1
- net /SERVO_PWM_1: track 0.00 -> 29.9 mm, vias 0 -> 1
- net /SERVO_PWM_4: track 0.00 -> 28.6 mm, vias 0 -> 1
- net /SERVO_PWM_2: track 0.00 -> 26.6 mm, vias 0 -> 1
- net +3V3: track 0.00 -> 24.6 mm, vias 0 -> 1
- net /Peripherals/BARO_I2C_SDA: track 0.00 -> 19.6 mm, vias 0 -> 1
- net /Peripherals/SD_CARD_SPI_MOSI: track 0.00 -> 19.5 mm, vias 0 -> 1
- net /RECEIVER_UART_RX: track 0.00 -> 18.0 mm, vias 0 -> 1
- net /Peripherals/SD_CARD_SPI_CLK: track 0.00 -> 17.2 mm, vias 0 -> 1
- net /Peripherals/BARO_I2C_SCL: track 0.00 -> 17.0 mm, vias 0 -> 1
- net /Peripherals/IMU_SPI_MISO: track 0.00 -> 16.8 mm, vias 0 -> 1
- net /COMP_I2C_SCL: track 0.00 -> 16.8 mm, vias 0 -> 1
- net /Peripherals/IMU_SPI_CS: track 0.00 -> 16.0 mm, vias 0 -> 1
- net /Peripherals/SD_CARD_SPI_MISO: track 0.00 -> 13.6 mm, vias 0 -> 1
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- added copper zone on B.Cu, net /ESC_BEC
- added copper zone on F.Cu, net /ESC_BEC
- added copper zone on F.Cu, net /ONBOARD_BEC
- added copper zone on F.Cu, net /SW
- added copper zone on F.Cu, net GND
- added copper zone on F.Cu, net VBAT

Commit message: More work
Parts:
- moved R8 0.68 mm to (40.3, 46.6)
- moved R9 0.68 mm to (38.8, 46.6)
- moved J2 0.50 mm to (31.8, 43.5)
- moved J3 0.50 mm to (30.5, 62.5)
- moved C9 0.23 mm to (45.0, 49.4)
- moved C13 0.09 mm to (41.5, 50.8)
Connections:
- J5 pad 1: /GPS_UART_TX -> GND
- J5 pad 2: /GPS_UART_RX -> +5V
- J5 pad 3: +5V -> /GPS_UART_RX
- J5 pad 4: GND -> /GPS_UART_TX
- J5 pad 5: /COMP_I2C_SDA -> /COMP_I2C_SCL
- J5 pad 6: /COMP_I2C_SCL -> /COMP_I2C_SDA
- J6 pad 1: /VTX_UART_TX -> VBAT
- J6 pad 2: /VTX_UART_RX -> GND
- J6 pad 3: VBAT_P -> /VTX_UART_TX
- J6 pad 4: GND -> /VTX_UART_RX
Routing:
- net +5V: track 7.91 -> 81.7 mm, vias 0 -> 3
- net VBAT: track 0.00 -> 54.1 mm, vias 0 -> 2
- net 5V_BEC: track 5.21 -> 46.0 mm
- net GND: track 4.10 -> 21.4 mm, vias 18 -> 62
- net /VTX_UART_TX: track 0.00 -> 9.15 mm, vias 0 -> 1
- net /VBAT_S: track 0.00 -> 8.45 mm, vias 0 -> 1
- net /VTX_UART_RX: track 0.00 -> 4.43 mm, vias 0 -> 1
- net /SERVO_PWM_4: track 28.6 -> 32.6 mm, vias 1 -> 0
- net /GPS_UART_TX: track 8.74 -> 5.75 mm
- net /SERVO_PWM_3: track 33.8 -> 36.7 mm, vias 1 -> 0
- net /COMP_I2C_SDA: track 13.3 -> 15.9 mm
- net /Peripherals/BARO_I2C_SCL: track 17.0 -> 19.5 mm
- net Net-(U3-BYPASS): track 0.00 -> 2.16 mm
- net /ESC_BEC: track 8.83 -> 6.68 mm, vias 3 -> 0
- net /SERVO_PWM_2: track 26.6 -> 28.5 mm, vias 1 -> 0
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- added copper zone on B.Cu, net GND
- removed copper zone on B.Cu, net /ESC_BEC
- removed copper zone on F.Cu, net /ESC_BEC
Other:
- board text added: "5V"
- board text added: "5x"
- board text added: "ESC PWM"
- board text added: "G"
- board text added: "GND"
- board text added: "GPS"
- board text added: "PWM"
- board text added: "PWM1"
- board text added: "PWM2"
- board text added: "PWM3"
- board text added: "PWM4"
- board text added: "RECV"
- board text added: "RX"
- board text added: "SCL"
- board text added: "SDA"
- board text added: "TX"
- board text added: "VBAT"
- board text added: "VTX"

Commit message: Finished PCB
Parts:
- J4, J6: footprint Connector_JST:JST_GH_SM04B-GHS-TB_1x04-1MP_P1.25mm_Horizontal -> toto_fc:4_pads
- J5: footprint Connector_JST:JST_GH_SM06B-GHS-TB_1x06-1MP_P1.25mm_Horizontal -> toto_fc:6_pads
- moved J5 5.59 mm to (56.0, 74.5), turned to 0 degrees
- moved J6 3.16 mm to (29.0, 83.0), turned to 0 degrees
- moved J4 2.42 mm to (56.0, 47.0), turned to 0 degrees
Connections:
- J4 pad 1: /RECEIVER_UART_TX -> GND
- J4 pad 2: /RECEIVER_UART_RX -> +5V
- J4 pad 3: +5V -> /RECEIVER_UART_TX
- J4 pad 4: GND -> /RECEIVER_UART_RX
- J5 pad 3: /GPS_UART_RX -> /GPS_UART_TX
- J5 pad 4: /GPS_UART_TX -> /GPS_UART_RX
- J6 pad 1: VBAT -> GND
- J6 pad 2: GND -> VBAT
Routing:
- net +5V: track 81.7 -> 73.3 mm
- net /COMP_I2C_SDA: track 15.9 -> 8.36 mm
- net /VTX_UART_RX: track 4.43 -> 8.46 mm
- net /RECEIVER_UART_RX: track 18.1 -> 14.6 mm
- net VBAT: track 54.1 -> 57.3 mm
- net /RECEIVER_UART_TX: track 13.3 -> 16.3 mm
- net /COMP_I2C_SCL: track 15.6 -> 13.1 mm
- net /GPS_UART_TX: track 5.75 -> 7.82 mm
- net /VTX_UART_TX: track 9.15 -> 8.13 mm
- net /GPS_UART_RX: track 7.13 -> 7.63 mm
- net GND: vias 62 -> 67
