File: pcb/toto_fc.kicad_sch (KiCad schematic)
At the start: 28 parts, among them J1 Battery Pads, J10 ESC PWM, J2 Debug Probe, J3 Receiver Pads, J4 GPS Pads, J5 VTX Pads, J6 Servo 1, J7 Servo 2, J8 Servo 3, J9 Servo 4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

Commit message: More pcb work
Parts:
- removed D1: PMEG2010EH, Diode_SMD:D_SOD-123F, symbol Diode:PMEG2010EH
- removed J1: Battery Pads, symbol Connector_Generic:Conn_01x03
- removed J10: ESC PWM, symbol Connector_Generic:Conn_01x01
- removed J2: Debug Probe, symbol Connector_Generic:Conn_01x04
- removed J6: Servo 1, symbol Connector_Generic:Conn_01x03
- removed J7: Servo 2, symbol Connector_Generic:Conn_01x03
- removed J8: Servo 3, symbol Connector_Generic:Conn_01x03
- removed J9: Servo 4, symbol Connector_Generic:Conn_01x03
- added C2: 100n, Capacitor_SMD:C_0603_1608Metric, symbol Device:C
- added J1: Conn_01x02, toto_fc:vbat_pads, symbol Connector_Generic:Conn_01x02
- added J2: Conn_01x12, toto_fc:pwm_headers, symbol Connector_Generic:Conn_01x12
- added J3: Conn_01x03, Connector_PinHeader_2.54mm:PinHeader_1x03_P2.54mm_Vertical, symbol Connector_Generic:Conn_01x03
- added J7: Conn_01x06_Shielded, symbol Connector_Generic_Shielded:Conn_01x06_Shielded
- added JP1: BEC_SJ, Jumper:SolderJumper-2_P1.3mm_Open_Pad1.0x1.5mm, symbol Jumper:SolderJumper_2_Bridged
- added JP2: ESC_SJ, Jumper:SolderJumper-2_P1.3mm_Open_Pad1.0x1.5mm, symbol Jumper:SolderJumper_2_Bridged
- C1: footprint (none) -> Capacitor_SMD:C_0805_2012Metric
- C3: renamed from C2; footprint (none) -> Capacitor_SMD:C_0805_2012Metric
- C4: renamed from C3; footprint (none) -> Capacitor_SMD:C_0603_1608Metric
- C5: renamed from C4; footprint (none) -> Capacitor_SMD:C_0805_2012Metric
- C6: renamed from C5; footprint (none) -> Capacitor_SMD:C_0805_2012Metric
- C7: renamed from C6; footprint (none) -> Capacitor_SMD:C_0603_1608Metric
- J4: renamed from J3; value Receiver Pads -> Receiver Connector; footprint (none) -> Connector_JST:JST_GH_BM04B-GHS-TBT_1x04-1MP_P1.25mm_Vertical
- J5: renamed from J4; value GPS Pads -> GPS Connector; footprint (none) -> Connector_JST:JST_GH_BM06B-GHS-TBT_1x06-1MP_P1.25mm_Vertical
- J6: renamed from J5; value VTX Pads -> VTX Connector; footprint (none) -> Connector_JST:JST_GH_BM04B-GHS-TBT_1x04-1MP_P1.25mm_Vertical
- L1: footprint (none) -> toto_fc:F1C2-060606W-5R6M
- R1, R2, R3, R4, R5, R6: footprint (none) -> Resistor_SMD:R_0603_1608Metric
- renumbered D2 to D1, D3 to D2
Connections:
- net 5V_BEC: now also J2.11 (Pin_11), J2.2 (Pin_2), J2.5 (Pin_5), J2.8 (Pin_8), JP1.2 (B), JP2.2 (B); no longer C5.1, C6.1, L1.2, R2.2, R4.2
- net COMP_I2C_SCL: now also J5.6 (Pin_6); no longer J5.5 (Pin_5)
- net COMP_I2C_SDA: now also J5.5 (Pin_5); no longer J5.6 (Pin_6)
- net ESC_PWM: now also J3.3 (Pin_3)
- net GND: now also C2.2, J1.2 (Pin_2), J2.1 (Pin_1), J2.10 (Pin_10), J2.4 (Pin_4), J2.7 (Pin_7), J3.1 (Pin_1)
- net SERVO_PWM_1: now also J2.3 (Pin_3)
- net SERVO_PWM_2: now also J2.6 (Pin_6)
- net SERVO_PWM_3: now also J2.9 (Pin_9)
- net SERVO_PWM_4: now also J2.12 (Pin_12)
- net VBAT: now also C2.1, J1.1 (Pin_1)
- net BOOT: now reaches C3.1, U1.4 (BOOT)
- net SWCLK: no longer names the net of A1.D1 (SWCLK)
- net SWDIO: no longer names the net of A1.D3 (SWDIO)
- new net ESC_BEC: J3.2 (Pin_2), JP2.1 (A)
- new net ONBOARD_BEC: C5.1, C6.1, JP1.1 (A), L1.2, R2.2, R4.2
- no-connect marks 5 -> 7
Other:
- note removed: "Skipped HF caps (doesn't apply for SMD afaik)"
- moved on the sheet: C1, C3, C4, C5, C6, D2, J4, J5, J6, L1, R1, R2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

Commit message: More work on the pcb
Parts:
- removed J7: Conn_01x06_Shielded, symbol Connector_Generic_Shielded:Conn_01x06_Shielded
- A1: footprint Module:RaspberryPi_Pico_SMD_HandSolder -> toto_fc:RaspberryPi_Pico_SMD_HandSolder
- J4, J6: footprint Connector_JST:JST_GH_BM04B-GHS-TBT_1x04-1MP_P1.25mm_Vertical -> Connector_JST:JST_GH_SM04B-GHS-TB_1x04-1MP_P1.25mm_Horizontal
- J5: footprint Connector_JST:JST_GH_BM06B-GHS-TBT_1x06-1MP_P1.25mm_Vertical -> Connector_JST:JST_GH_SM06B-GHS-TB_1x06-1MP_P1.25mm_Horizontal
Connections:
- net GND: now also J2.12 (Pin_12), J2.3 (Pin_3), J2.6 (Pin_6), J2.9 (Pin_9); no longer J2.1 (Pin_1), J2.10 (Pin_10), J2.4 (Pin_4), J2.7 (Pin_7)
- net SERVO_PWM_1: now also J2.1 (Pin_1); no longer J2.3 (Pin_3)
- net SERVO_PWM_2: now also J2.4 (Pin_4); no longer J2.6 (Pin_6)
- net SERVO_PWM_3: now also J2.7 (Pin_7); no longer J2.9 (Pin_9)
- net SERVO_PWM_4: now also J2.10 (Pin_10); no longer J2.12 (Pin_12)

Commit message: more progress
Parts:
- removed D1: PESD1IVN27-AX, Diode_SMD:D_SOD-323F, symbol Device:D_TVS
- added CR1: D24V0S1U2TQ-7, toto_fc:SOD523, symbol toto_fc:D24V0S1U2TQ-7
Connections:
- net GND: now also CR1.2
- net VBAT: now also CR1.1
Changed lines of the file:
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@@
-	(wire
-		(pts
-			(xy 153.67 45.72) (xy 153.67 52.07)
-		)
-		(stroke
-			(width 0)
-			(type default)
-		)
-	)
 	(wire
 		(pts
@@
 	(wire
 		(pts
-			(xy 153.67 33.02) (xy 153.67 38.1)
+			(xy 153.67 33.02) (xy 153.67 36.83)
 		)
 		(stroke
@@
 		(pts
 			(xy 242.57 129.54) (xy 256.54 129.54)
+		)
+		(stroke
+			(width 0)
+			(type default)
+		)
+	)
+	(wire
+		(pts
+			(xy 153.67 46.99) (xy 153.67 52.07)
 		)
 		(stroke
@@
 			)
 			(justify left bottom)
-		)
-	)
-	(symbol
-		(lib_id "Device:D_TVS")
-		(at 153.67 41.91 90)
-		(unit 1)
-		(exclude_from_sim no)
-		(in_bom yes)
-		(on_board yes)
-		(dnp no)
-		(fields_autoplaced yes)
-		(property "Reference" "D1"
-			(at 156.21 40.6399 90)
-			(effects
-				(font
-					(size 1.27 1.27)
-				)
-				(justify right)
-			)
-		)
-		(property "Value" "PESD1IVN27-AX"
-			(at 156.21 43.1799 90)
-			(effects
-				(font
-					(size 1.27 1.27)
-				)
-				(justify right)
-			)
-		)
-		(property "Footprint" "Diode_SMD:D_SOD-323F"
-			(at 153.67 41.91 0)
-			(effects
-				(font
-					(size 1.27 1.27)
-				)
-				(hide yes)
-			)
-		)
-		(property "Datasheet" "~"
-			(at 153.67 41.91 0)
-			(effects
-				(font
-					(size 1.27 1.27)
-				)
-				(hide yes)
-			)
-		)
-		(property "Description" "Bidirectional transient-voltage-suppression diode"
-			(at 153.67 41.91 0)
-			(effects
-				(font
-					(size 1.27 1.27)
-				)
-				(hide yes)
-			)
-		)
-		(pin "1"
-		)
-		(pin "2"
-		)
-		(instances
-			(project "toto_fc"
-				(path "/0259efb7-694a-4ce2-9998-fdf65c8a3c90"
-					(reference "D1")
-					(unit 1)
-				)
-			)
 		)
 	)
@@
 					(unit 1)
 				)
+			)
+		)
+	)
+	(symbol
+		(lib_id "toto_fc:D24V0S1U2TQ-7")
+		(at 153.67 46.99 90)
+		(unit 1)
+		(exclude_from_sim no)
+		(in_bom yes)
+		(on_board yes)
+		(dnp no)
+		(fields_autoplaced yes)
+		(property "Reference" "CR1"
+			(at 157.48 40.6399 90)
+			(effects
+				(font
+					(size 1.524 1.524)
+				)
+				(justify right)
+			)
+		)
+		(property "Value" "D24V0S1U2TQ-7"
+			(at 157.48 43.1799 90)
+			(effects
+				(font
+					(size 1.524 1.524)
+				)
+				(justify right)
+			)
+		)
+		(property "Footprint" "toto_fc:SOD523"
+			(at 153.67 46.99 0)
+			(effects
+				(font
+					(size 1.27 1.27)
+					(italic yes)
+				)
+				(hide yes)
+			)
+		)
+		(property "Datasheet" "D24V0S1U2TQ-7"
+			(at 153.67 46.99 0)
+			(effects
+				(font
+					(size 1.27 1.27)
+					(italic yes)
+				)
+				(hide yes)
+			)
+		)
+		(property "Description" ""
+			(at 153.67 46.99 0)
+			(effects
+				(font
+					(size 1.27 1.27)
+				)
+				(hide yes)
+			)
+		)
+		(pin "1"
+		)
+		(pin "2"
+		)
+		(instances
+			(project ""
+				(path "/0259efb7-694a-4ce2-9998-fdf65c8a3c90"
+					(reference "CR1")
+					(unit 1)
+				)

Commit message: More work
Connections:
- net VBAT_P is gone; now on net VTX_UART_TX: J6.3 (Pin_3)
- net +5V: now also J5.2 (Pin_2); no longer J5.3 (Pin_3)
- net COMP_I2C_SCL: now also J5.5 (Pin_5); no longer J5.6 (Pin_6)
- net COMP_I2C_SDA: now also J5.6 (Pin_6); no longer J5.5 (Pin_5)
- net GND: now also J5.1 (Pin_1), J6.2 (Pin_2); no longer J5.4 (Pin_4), J6.4 (Pin_4)
- net GPS_UART_RX: now also J5.3 (Pin_3); no longer J5.2 (Pin_2)
- net GPS_UART_TX: now also J5.4 (Pin_4); no longer J5.1 (Pin_1)
- net VBAT: now also J6.1 (Pin_1)
- net VTX_UART_RX: now also J6.4 (Pin_4); no longer J6.2 (Pin_2)
- net VTX_UART_TX: no longer J6.1 (Pin_1)
Other:
- moved on the sheet: CR1, D2

Commit message: Finished PCB
Parts:
- J4, J6: footprint Connector_JST:JST_GH_SM04B-GHS-TB_1x04-1MP_P1.25mm_Horizontal -> toto_fc:4_pads
- J5: footprint Connector_JST:JST_GH_SM06B-GHS-TB_1x06-1MP_P1.25mm_Horizontal -> toto_fc:6_pads
Connections:
- net +5V: now also J4.2 (Pin_2); no longer J4.3 (Pin_3)
- net GND: now also J4.1 (Pin_1), J6.1 (Pin_1); no longer J4.4 (Pin_4), J6.2 (Pin_2)
- net GPS_UART_RX: now also J5.4 (Pin_4); no longer J5.3 (Pin_3)
- net GPS_UART_TX: now also J5.3 (Pin_3); no longer J5.4 (Pin_4)
- net RECEIVER_UART_RX: now also J4.4 (Pin_4); no longer J4.2 (Pin_2)
- net RECEIVER_UART_TX: now also J4.3 (Pin_3); no longer J4.1 (Pin_1)
- net VBAT: now also J6.2 (Pin_2); no longer J6.1 (Pin_1)
Changed lines of the file:
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@@
 	(wire
 		(pts
+			(xy 242.57 106.68) (xy 256.54 106.68)
+		)
+		(stroke
+			(width 0)
+			(type default)
+		)
+	)
+	(wire
+		(pts
 			(xy 54.61 152.4) (xy 54.61 156.21)
 		)
@@
 	(wire
 		(pts
-			(xy 125.73 64.77) (xy 113.03 64.77)
+			(xy 243.84 127) (xy 256.54 127)
 		)
 		(stroke
@@
 	(wire
 		(pts
-			(xy 243.84 124.46) (xy 256.54 124.46)
+			(xy 125.73 64.77) (xy 113.03 64.77)
 		)
 		(stroke
@@
 	(wire
 		(pts
+			(xy 238.76 111.76) (xy 256.54 111.76)
+		)
+		(stroke
+			(width 0)
+			(type default)
+		)
+	)
+	(wire
+		(pts
+			(xy 241.3 105.41) (xy 242.57 105.41)
+		)
+		(stroke
+			(width 0)
+			(type default)
+		)
+	)
+	(wire
+		(pts
 			(xy 95.25 163.83) (xy 104.14 163.83)
 		)
@@
 	(wire
 		(pts
+			(xy 238.76 109.22) (xy 256.54 109.22)
+		)
+		(stroke
+			(width 0)
+			(type default)
+		)
+	)
+	(wire
+		(pts
 			(xy 242.57 129.54) (xy 256.54 129.54)
 		)
@@
 	(wire
 		(pts
-			(xy 243.84 127) (xy 256.54 127)
-		)
-		(stroke
-			(width 0)
-			(type default)
-		)
-	)
-	(wire
-		(pts
 			(xy 101.6 157.48) (xy 109.22 157.48)
 		)
@@
 	(wire
 		(pts
-			(xy 238.76 104.14) (xy 256.54 104.14)
-		)
-		(stroke
-			(width 0)
-			(type default)
-		)
-	)
-	(wire
-		(pts
 			(xy 120.65 87.63) (xy 113.03 87.63)
 		)
@@
 	(wire
 		(pts
+			(xy 242.57 105.41) (xy 242.57 106.68)
+		)
+		(stroke
+			(width 0)
+			(type default)
+		)
+	)
+	(wire
+		(pts
 			(xy 187.96 130.81) (xy 212.09 130.81)
 		)
@@
 	(wire
 		(pts
+			(xy 242.57 104.14) (xy 256.54 104.14)
+		)
+		(stroke
+			(width 0)
+			(type default)
+		)
+	)
+	(wire
+		(pts
 			(xy 149.86 167.64) (xy 149.86 166.37)
 		)
@@
 	(wire
 		(pts
+			(xy 242.57 102.87) (xy 242.57 104.14)
+		)
+		(stroke
+			(width 0)
+			(type default)
+		)
+	)
+	(wire
+		(pts
+			(xy 242.57 102.87) (xy 241.3 102.87)
+		)
+		(stroke
+			(width 0)
+			(type default)
+		)
+	)
+	(wire
+		(pts
 			(xy 54.61 156.21) (xy 58.42 156.21)
 		)
@@
 	(wire
 		(pts
-			(xy 238.76 106.68) (xy 256.54 106.68)
+			(xy 49.53 77.47) (xy 67.31 77.47)
 		)
 		(stroke
@@
 	(wire
 		(pts
-			(xy 49.53 77.47) (xy 67.31 77.47)
+			(xy 46.99 67.31) (xy 67.31 67.31)
 		)
 		(stroke
@@
 	(wire
 		(pts
-			(xy 46.99 67.31) (xy 67.31 67.31)
+			(xy 194.31 40.64) (xy 196.85 40.64)
 		)
 		(stroke
@@
 	(wire
 		(pts
-			(xy 194.31 40.64) (xy 196.85 40.64)
+			(xy 118.11 182.88) (xy 118.11 181.61)
 		)
 		(stroke
@@
 	(wire
 		(pts
-			(xy 118.11 182.88) (xy 118.11 181.61)
+			(xy 243.84 124.46) (xy 256.54 124.46)
 		)
 		(stroke
@@
 		)
 	)
-	(label "GPS_UART_TX"
-		(at 243.84 127 0)
+	(label "VBAT_S"
+		(at 220.98 40.64 180)
 		(effects
 			(font
 				(size 1.27 1.27)
 			)
-			(justify left bottom)
+			(justify right bottom)
 		)
 	)
-	(label "RECEIVER_UART_TX"
-		(at 238.76 104.14 0)
+	(label "RECEIVER_UART_RX"
+		(at 238.76 111.76 0)
 		(effects
 			(font
@@
 		)
 	)
-	(label "VBAT_S"
-		(at 220.98 40.64 180)
-		(effects
-			(font
-				(size 1.27 1.27)
-			)
-			(justify right bottom)
-		)
-	)
 	(label "COMP_I2C_SCL"
 		(at 242.57 129.54 0)
@@
 		)
 	)
+	(label "GPS_UART_TX"
+		(at 243.84 124.46 0)
+		(effects
+			(font
+				(size 1.27 1.27)
+			)
+			(justify left bottom)
+		)
+	)
 	(label "ONBOARD_BEC"
 		(at 137.16 157.48 0)
@@
 		)
 	)
-	(label "GPS_UART_RX"
-		(at 243.84 124.46 0)
-		(effects
-			(font
-				(size 1.27 1.27)
-			)
-			(justify left bottom)
-		)
-	)
 	(label "RECEIVER_UART_RX"
 		(at 49.53 77.47 0)
@@
 		)
 	)
+	(label "GPS_UART_RX"
+		(at 243.84 127 0)
+		(effects
+			(font
+				(size 1.27 1.27)
+			)
+			(justify left bottom)
+		)
+	)
 	(label "COMP_I2C_SDA"
 		(at 53.34 95.25 0)
@@
 		)
 	)
-	(label "RECEIVER_UART_RX"
-		(at 238.76 106.68 0)
-		(effects
-			(font
-				(size 1.27 1.27)
-			)
-			(justify left bottom)
-		)
-	)
 	(label "SERVO_PWM_3"
 		(at 127 72.39 180)
@@
 		)
 	)
+	(label "RECEIVER_UART_TX"
+		(at 238.76 109.22 0)
+		(effects
+			(font
+				(size 1.27 1.27)
+			)
+			(justify left bottom)
+		)
+	)
 	(label "VTX_UART_TX"
 		(at 125.73 62.23 180)
@@
 			)
 		)
-		(property "Footprint" "Connector_JST:JST_GH_SM06B-GHS-TB_1x06-1MP_P1.25mm_Horizontal"
+		(property "Footprint" "toto_fc:6_pads"
 			(at 261.62 124.46 0)
 			(effects
@@
 	(symbol
 		(lib_id "power:+5V")
-		(at 256.54 109.22 90)
+		(at 241.3 105.41 90)
 		(unit 1)
 		(exclude_from_sim no)
@@
 		(fields_autoplaced yes)
 		(property "Reference" "#PWR027"
-			(at 260.35 109.22 0)
+			(at 245.11 105.41 0)
 			(effects
 				(font
@@
 		)
 		(property "Value" "+5V"
-			(at 252.73 109.2199 90)
+			(at 237.49 105.4099 90)
 			(effects
 				(font
@@
 		)
 		(property "Footprint" ""
-			(at 256.54 109.22 0)
+			(at 241.3 105.41 0)
 			(effects
 				(font
@@
 		)
 		(property "Datasheet" ""
-			(at 256.54 109.22 0)
+			(at 241.3 105.41 0)
 			(effects
 				(font
@@
 		)
 		(property "Description" "Power symbol creates a global label with name \"+5V\""
-			(at 256.54 109.22 0)
+			(at 241.3 105.41 0)
 			(effects
 				(font
@@
 	(symbol
 		(lib_id "toto_fc:VBAT")
-		(at 241.3 139.7 90)
+		(at 241.3 142.24 90)
 		(unit 1)
 		(exclude_from_sim no)
@@
 		(fields_autoplaced yes)
 		(property "Reference" "#PWR024"
-			(at 245.11 139.7 0)
+			(at 245.11 142.24 0)
 			(effects
 				(font
@@
 		)
 		(property "Value" "VBAT"
-			(at 237.49 139.6999 90)
+			(at 237.49 142.2399 90)
 			(effects
 				(font
@@
 		)
 		(property "Footprint" ""
-			(at 241.3 139.7 0)
+			(at 241.3 142.24 0)
 			(effects
 				(font
@@
 		)
 		(property "Datasheet" ""
-			(at 241.3 139.7 0)
+			(at 241.3 142.24 0)
 			(effects
 				(font
@@
 		)
 		(property "Description" "Power symbol creates a global label with name {dblquote}VBAT{dblquote}"
-			(at 241.3 139.7 0)
+			(at 241.3 142.24 0)
 			(effects
 				(font
@@
 			)
 		)
-		(property "Footprint" "Connector_JST:JST_GH_SM04B-GHS-TB_1x04-1MP_P1.25mm_Horizontal"
+		(property "Footprint" "toto_fc:4_pads"
 			(at 261.62 142.24 0)
 			(effects
@@
 	(symbol
 		(lib_id "power:GND")
-		(at 241.3 142.24 270)
+		(at 241.3 139.7 270)
 		(unit 1)
 		(exclude_from_sim no)
@@
 		(fields_autoplaced yes)
 		(property "Reference" "#PWR025"
-			(at 234.95 142.24 0)
+			(at 234.95 139.7 0)
 			(effects
 				(font
@@
 		)
 		(property "Value" "GND"
-			(at 237.49 142.2399 90)
+			(at 237.49 139.6999 90)
 			(effects
 				(font
@@
 		)
 		(property "Footprint" ""
-			(at 241.3 142.24 0)
+			(at 241.3 139.7 0)
 			(effects
 				(font
@@
 		)
 		(property "Datasheet" ""
-			(at 241.3 142.24 0)
+			(at 241.3 139.7 0)
 			(effects
 				(font
@@
 		)
 		(property "Description" "Power symbol creates a global label with name \"GND\" , ground"
-			(at 241.3 142.24 0)
+			(at 241.3 139.7 0)
 			(effects
 				(font
@@
 			)
 		)
-		(property "Footprint" "Connector_JST:JST_GH_SM04B-GHS-TB_1x04-1MP_P1.25mm_Horizontal"
+		(property "Footprint" "toto_fc:4_pads"
 			(at 261.62 106.68 0)
 			(effects
@@
 	(symbol
 		(lib_id "power:GND")
-		(at 256.54 111.76 270)
+		(at 241.3 102.87 270)
 		(unit 1)
 		(exclude_from_sim no)
@@
 		(fields_autoplaced yes)
 		(property "Reference" "#PWR028"
-			(at 250.19 111.76 0)
+			(at 234.95 102.87 0)
 			(effects
 				(font
@@
 		)
 		(property "Value" "GND"
-			(at 252.73 111.7599 90)
+			(at 237.49 102.8699 90)
 			(effects
 				(font
@@
 		)
 		(property "Footprint" ""
-			(at 256.54 111.76 0)
+			(at 241.3 102.87 0)
 			(effects
 				(font
@@
 		)
 		(property "Datasheet" ""
-			(at 256.54 111.76 0)
+			(at 241.3 102.87 0)
 			(effects
 				(font
@@
 		)
 		(property "Description" "Power symbol creates a global label with name \"GND\" , ground"
-			(at 256.54 111.76 0)
+			(at 241.3 102.87 0)
 			(effects
 				(font
